File: hardware/GameConsole_ESP32.kicad_pcb (KiCad board)
At the start: 2 copper layers, 82 x 85 mm, 17 parts, among them J1 Conn_01x20_Socket, J2 Conn_01x20_Socket, SW1 RedBtn, SW2 GreenBtn, SW3 YellowBtn, SW4 BlueBtn, U1 I2C OLED

Commit message: Cleaned up schematic and updated PCB design
Parts:
- added REF**: MountingHole_3.2mm_M3, MountingHole:MountingHole_3.2mm_M3, F.Cu at (111.2, 44.3)
- added REF**: MountingHole_3.2mm_M3, MountingHole:MountingHole_3.2mm_M3, F.Cu at (181.1, 44.1)
- moved J3 1.00 mm to (109.0, 117.1)
- moved J2 0.87 mm to (120.7, 66.0)
- moved J1 0.82 mm to (169.0, 40.6)
- renumbered Blue to Blue1, Green to Green1, Joystick to J3, Red to Red1, Yellow to Yellow1
Connections:
- net /14 renamed /BZR
- net /16 renamed /BTN_Blue
- net /17 renamed /LED_Blue
- net /18 renamed /LED_Red
- net /19 renamed /LED_Green
- net /21 renamed /I2C_SDA
- net /22 renamed /I2C_SCL
- net /25 renamed /BTN_Green
- net /26 renamed /BTN_Red
- net /27 renamed /BTN_Yellow
- net /32 renamed /SW
- net /34 renamed /VRx
- net /35 renamed /VRy
- net Net-(J1-Pin_13) renamed /LED_Yellow
- J1 pad 1: /3.3V -> unconnected-(J1-Pin_1-Pad1)
- J1 pad 16: unconnected-(J1-Pin_16-Pad16) -> +3V3
- J1 pad 17: unconnected-(J1-Pin_17-Pad17) -> +3V3
- J1 pad 18: /3.3V -> +3V3
- J3 pad 4: /3.3V -> +3V3
- U1 pad 2: /3.3V -> +3V3
Routing:
- net /3.3V: track 122.2 -> 0.00 mm, vias 1 -> 0
- net +3V3: track 0.00 -> 115.5 mm, vias 0 -> 1
- net /BZR: track 68.3 -> 62.2 mm
- net /BTN_Yellow: track 96.2 -> 93.7 mm
- net /SW: track 123.5 -> 121.9 mm
- net /BTN_Red: track 80.1 -> 80.9 mm
- net /BTN_Green: track 93.8 -> 94.5 mm
- net /VRy: track 122.3 -> 121.7 mm
Other:
- board text added: "Game Console V1.0"
- board text removed: "Game Console"
